Commit message: Added gazebo functionality

File: description/robot_core.xacro (robot description, xacro)
@@ -41,4 +41,7 @@
         </xacro:inertial_box>
     </link>
+    <gazebo reference="chassis">
+        <material>Gazebo/White</material>
+    </gazebo>
     <!-- Left Wheel Link-->
     <joint name="left_wheel_joint" type="continuous">
@@ -51,5 +54,5 @@
         <visual>
             <geometry>
-                <cylinder radius="0.05" length="0.04"/>
+                <cylinder radius="0.0325" length="0.04"/>
             </geometry>
             <material name="blue"/>
@@ -57,11 +60,14 @@
         <collision>
             <geometry>
-                <cylinder radius="0.05" length="0.04"/>
+                <cylinder radius="0.0325" length="0.04"/>
             </geometry>
         </collision>
-        <xacro:inertial_cylinder mass ="0.1" length = "0.04" radius = "0.05">
+        <xacro:inertial_cylinder mass ="0.1" length = "0.04" radius = "0.0325">
             <origin xyz = "0 0 0" rpy = "0 0 0"/>
         </xacro:inertial_cylinder>
     </link>
+    <gazebo reference="left_wheel">
+        <material>Gazebo/Blue</material>
+    </gazebo>
     <!-- Right Wheel Link-->
     <joint name="right_wheel_joint" type="continuous">
@@ -74,5 +80,5 @@
         <visual>
             <geometry>
-                <cylinder radius="0.05" length="0.04"/>
+                <cylinder radius="0.0325" length="0.04"/>
             </geometry>
             <material name="blue"/>
@@ -80,11 +86,14 @@
         <collision>
             <geometry>
-                <cylinder radius="0.05" length="0.04"/>
+                <cylinder radius="0.0325" length="0.04"/>
             </geometry>
         </collision>
-        <xacro:inertial_cylinder mass ="0.1" length = "0.04" radius = "0.05">
+        <xacro:inertial_cylinder mass ="0.1" length = "0.04" radius = "0.0325">
             <origin xyz = "0 0 0" rpy = "0 0 0"/>
         </xacro:inertial_cylinder>
     </link>
+    <gazebo reference="right_wheel">
+        <material>Gazebo/Blue</material>
+    </gazebo>
     <!--Caster wheel link-->
     <joint name="caster_wheel_joint" type="fixed">
@@ -96,5 +105,5 @@
         <visual>
             <geometry>
-                <sphere radius="0.05"/>
+                <sphere radius="0.0325"/>
             </geometry>
             <material name="black"/>
@@ -102,10 +111,15 @@
         <collision>
             <geometry>
-                <sphere radius="0.05"/>
+                <sphere radius="0.0325"/>
             </geometry>
         </collision>
-        <xacro:inertial_sphere mass ="0.1" radius = "0.05">
+        <xacro:inertial_sphere mass ="0.1" radius = "0.0325">
             <origin xyz = "0 0 0" rpy = "0 0 0"/>
         </xacro:inertial_sphere>
     </link>
+    <gazebo reference="caster_wheel">
+        <material>Gazebo/Black</material>
+        <mu1 value="0.001"/>
+        <mu2 value="0.002"/>
+    </gazebo>
 </robot>
